Commit message: feat: add collision and inertial

File: src/robot_description/urdf/robot.urdf.xacro (robot description, xacro)
@@ -3,23 +3,117 @@
     xmlns:xacro="http://www.ros.org/wiki/xacro"
     name="virtual_mobile_robot">
+    <!-- ================================================== -->
+    <!-- Parameters                                         -->
+    <!-- ================================================== -->
     <!-- Base -->
-    <xacro:property name="base_length" value="0.5" />
-    <xacro:property name="base_width" value="0.3" />
-    <xacro:property name="base_height" value="0.15" />
+    <xacro:property name="base_length" value="0.5"/>
+    <xacro:property name="base_width" value="0.3"/>
+    <xacro:property name="base_height" value="0.15"/>
+    <xacro:property name="base_mass" value="5.0"/>
     <!-- Wheels -->
-    <xacro:property name="wheel_radius" value="0.08" />
-    <xacro:property name="wheel_width" value="0.04" />
-    <xacro:property name="wheel_separation" value="0.34" />
-    <xacro:property name="wheel_x_offset" value="0.0" />
+    <xacro:property name="wheel_radius" value="0.08"/>
+    <xacro:property name="wheel_width" value="0.04"/>
+    <xacro:property name="wheel_separation" value="0.34"/>
+    <xacro:property name="wheel_x_offset" value="0.0"/>
+    <xacro:property name="wheel_mass" value="0.5"/>
     <!-- Lidar -->
-    <xacro:property name="lidar_radius" value="0.05" />
-    <xacro:property name="lidar_height" value="0.04" />
-    <xacro:property name="lidar_x_offset" value="0.15" />
-    <xacro:property name="lidar_z_offset" value="0.25" />
+    <xacro:property name="lidar_radius" value="0.05"/>
+    <xacro:property name="lidar_height" value="0.04"/>
+    <xacro:property name="lidar_x_offset" value="0.15"/>
+    <xacro:property name="lidar_z_offset" value="0.25"/>
+    <xacro:property name="lidar_mass" value="0.2"/>
+    <!--
+        base_link 位于地面中心附近。
+        轮子中心高度：
+        wheel_radius = 0.08
+        车体中心高度：
+        wheel_radius + base_height / 2
+        = 0.08 + 0.075
+        = 0.155
+    -->
+    <xacro:property
+        name="base_center_z"
+        value="${wheel_radius + base_height / 2.0}"/>
+    <!-- ================================================== -->
+    <!-- Inertial Macros                                    -->
+    <!-- ================================================== -->
+    <!--
+        长方体惯性宏
+        x: X 方向长度
+        y: Y 方向宽度
+        z: Z 方向高度
+    -->
+    <xacro:macro
+        name="box_inertial"
+        params="mass x y z origin_xyz">
+        <inertial>
+            <origin
+                xyz="${origin_xyz}"
+                rpy="0.0 0.0 0.0"/>
+            <mass value="${mass}"/>
+            <inertia
+                ixx="${mass * (y * y + z * z) / 12.0}"
+                ixy="0.0"
+                ixz="0.0"
+                iyy="${mass * (x * x + z * z) / 12.0}"
+                iyz="0.0"
+                izz="${mass * (x * x + y * y) / 12.0}"/>
+        </inertial>
+    </xacro:macro>
+    <!--
+        Y 轴圆柱惯性宏
+        适用于左右轮。
+        圆柱轴线沿 Y 轴。
+    -->
+    <xacro:macro
+        name="cylinder_inertial_y"
+        params="mass radius length origin_xyz">
+        <inertial>
+            <origin
+                xyz="${origin_xyz}"
+                rpy="0.0 0.0 0.0"/>
+            <mass value="${mass}"/>
+            <inertia
+                ixx="${mass * (3.0 * radius * radius + length * length) / 12.0}"
+                ixy="0.0"
+                ixz="0.0"
+                iyy="${mass * radius * radius / 2.0}"
+                iyz="0.0"
+                izz="${mass * (3.0 * radius * radius + length * length) / 12.0}"/>
+        </inertial>
+    </xacro:macro>
+    <!--
+        Z 轴圆柱惯性宏
+        适用于激光雷达外壳。
+        圆柱轴线沿 Z 轴。
+    -->
+    <xacro:macro
+        name="cylinder_inertial_z"
+        params="mass radius length origin_xyz">
+        <inertial>
+            <origin
+                xyz="${origin_xyz}"
+                rpy="0.0 0.0 0.0"/>
+            <mass value="${mass}"/>
+            <inertia
+                ixx="${mass * (3.0 * radius * radius + length * length) / 12.0}"
+                ixy="0.0"
+                ixz="0.0"
+                iyy="${mass * (3.0 * radius * radius + length * length) / 12.0}"
+                iyz="0.0"
+                izz="${mass * radius * radius / 2.0}"/>
+        </inertial>
+    </xacro:macro>
+    <!-- ================================================== -->
+    <!-- Base Link                                          -->
+    <!-- ================================================== -->
     <link name="base_link">
         <visual>
-            <origin xyz="0.0 0.0 ${wheel_radius + base_height / 2.0}" rpy="0.0 0.0 0.0"/>
-            <geometry>
-                <box size="${base_length} ${base_width} ${base_height}"/>
+            <origin
+                xyz="0.0 0.0 ${base_center_z}"
+                rpy="0.0 0.0 0.0"/>
+            <geometry>
+                <box
+                    size="${base_length} ${base_width} ${base_height}"/>
             </geometry>
             <material name="gray">
@@ -27,29 +121,88 @@
             </material>
         </visual>
+        <collision>
+            <origin
+                xyz="0.0 0.0 ${base_center_z}"
+                rpy="0.0 0.0 0.0"/>
+            <geometry>
+                <box
+                    size="${base_length} ${base_width} ${base_height}"/>
+            </geometry>
+        </collision>
+        <xacro:box_inertial
+            mass="${base_mass}"
+            x="${base_length}"
+            y="${base_width}"
+            z="${base_height}"
+            origin_xyz="0.0 0.0 ${base_center_z}"/>
     </link>
+    <!-- ================================================== -->
+    <!-- Wheel Macro                                        -->
+    <!-- ================================================== -->
     <xacro:macro name="wheel" params="name y_position">
         <link name="${name}_wheel_link">
             <visual>
-                <origin xyz="0.0 0.0 0.0" rpy="1.5708 0.0 0.0"/>
+                <!--
+                    URDF 中圆柱默认沿 Z 轴。
+                    绕 X 轴旋转 90 度后，
+                    圆柱轴变为沿 Y 轴。
+                -->
+                <origin
+                    xyz="0.0 0.0 0.0"
+                    rpy="${pi / 2.0} 0.0 0.0"/>
                 <geometry>
-                    <cylinder radius="${wheel_radius}" length="${wheel_width}"/>
+                    <cylinder
+                        radius="${wheel_radius}"
+                        length="${wheel_width}"/>
                 </geometry>
-                <material name="black">
+                <material name="${name}_wheel_black">
                     <color rgba="0.05 0.05 0.05 1.0"/>
                 </material>
             </visual>
+            <collision>
+                <origin
+                    xyz="0.0 0.0 0.0"
+                    rpy="${pi / 2.0} 0.0 0.0"/>
+                <geometry>
+                    <cylinder
+                        radius="${wheel_radius}"
+                        length="${wheel_width}"/>
+                </geometry>
+            </collision>
+            <xacro:cylinder_inertial_y
+                mass="${wheel_mass}"
+                radius="${wheel_radius}"
+                length="${wheel_width}"
+                origin_xyz="0.0 0.0 0.0"/>
         </link>
-        <joint name="${name}_wheel_joint" type="fixed">
+        <joint name="${name}_wheel_joint" type="continuous">
             <parent link="base_link"/>
             <child link="${name}_wheel_link"/>
-            <origin xyz="${wheel_x_offset} ${y_position} ${wheel_radius}" rpy="0.0 0.0 0.0"/>
+            <origin
+                xyz="${wheel_x_offset} ${y_position} ${wheel_radius}"
+                rpy="0.0 0.0 0.0"/>
+            <axis xyz="0.0 1.0 0.0"/>
         </joint>
     </xacro:macro>
-    <xacro:wheel name="left" y_position="${wheel_separation / 2.0}"/>
-    <xacro:wheel name="right" y_position="${-wheel_separation / 2.0}"/>
+    <!-- Left wheel -->
+    <xacro:wheel
+        name="left"
+        y_position="${wheel_separation / 2.0}"/>
+    <!-- Right wheel -->
+    <xacro:wheel
+        name="right"
+        y_position="${-wheel_separation / 2.0}"/>
+    <!-- ================================================== -->
+    <!-- Lidar                                              -->
+    <!-- ================================================== -->
     <link name="laser_frame">
         <visual>
-            <geometry>
-                <cylinder radius="${lidar_radius}" length="${lidar_height}"/>
+            <origin
+                xyz="0.0 0.0 0.0"
+                rpy="0.0 0.0 0.0"/>
+            <geometry>
+                <cylinder
+                    radius="${lidar_radius}"
+                    length="${lidar_height}"/>
             </geometry>
             <material name="blue">
@@ -57,9 +210,26 @@
             </material>
         </visual>
+        <collision>
+            <origin
+                xyz="0.0 0.0 0.0"
+                rpy="0.0 0.0 0.0"/>
+            <geometry>
+                <cylinder
+                    radius="${lidar_radius}"
+                    length="${lidar_height}"/>
+            </geometry>
+        </collision>
+        <xacro:cylinder_inertial_z
+            mass="${lidar_mass}"
+            radius="${lidar_radius}"
+            length="${lidar_height}"
+            origin_xyz="0.0 0.0 0.0"/>
     </link>
     <joint name="laser_joint" type="fixed">
         <parent link="base_link"/>
         <child link="laser_frame"/>
-        <origin xyz="${lidar_x_offset} 0 ${lidar_z_offset}" rpy="0.0 0.0 0.0"/>
+        <origin
+            xyz="${lidar_x_offset} 0.0 ${lidar_z_offset}"
+            rpy="0.0 0.0 0.0"/>
     </joint>
 </robot>

Commit message: feat: add swivel caster

File: src/robot_description/urdf/robot.urdf.xacro (robot description, xacro)
@@ -15,6 +15,10 @@
     <xacro:property name="wheel_width" value="0.04"/>
     <xacro:property name="wheel_separation" value="0.34"/>
-    <xacro:property name="wheel_x_offset" value="0.0"/>
+    <xacro:property name="wheel_x_offset" value="0.05"/>
     <xacro:property name="wheel_mass" value="0.5"/>
+    <!-- Caster wheel -->
+    <xacro:property name="caster_radius" value="0.04"/>
+    <xacro:property name="caster_x_offset" value="-0.20"/>
+    <xacro:property name="caster_mass" value="0.1"/>
     <!-- Lidar -->
     <xacro:property name="lidar_radius" value="0.05"/>
@@ -103,4 +107,25 @@
                 iyz="0.0"
                 izz="${mass * radius * radius / 2.0}"/>
+        </inertial>
+    </xacro:macro>
+    <!--
+    万向轮惯性宏
+    Sphere inertial macro
+    -->
+    <xacro:macro
+        name="sphere_inertial"
+        params="mass radius origin_xyz">
+        <inertial>
+            <origin
+                xyz="${origin_xyz}"
+                rpy="0.0 0.0 0.0"/>
+            <mass value="${mass}"/>
+            <inertia
+                ixx="${2.0 * mass * radius * radius / 5.0}"
+                ixy="0.0"
+                ixz="0.0"
+                iyy="${2.0 * mass * radius * radius / 5.0}"
+                iyz="0.0"
+                izz="${2.0 * mass * radius * radius / 5.0}"/>
         </inertial>
     </xacro:macro>
@@ -193,4 +218,39 @@
         name="right"
         y_position="${-wheel_separation / 2.0}"/>
+<!-- ================================================== -->
+<!-- Rear caster wheel                                  -->
+<!-- ================================================== -->
+<link name="caster_link">
+    <visual>
+        <origin
+            xyz="0.0 0.0 0.0"
+            rpy="0.0 0.0 0.0"/>
+        <geometry>
+            <sphere radius="${caster_radius}"/>
+        </geometry>
+        <material name="caster_gray">
+            <color rgba="0.25 0.25 0.25 1.0"/>
+        </material>
+    </visual>
+    <collision>
+        <origin
+            xyz="0.0 0.0 0.0"
+            rpy="0.0 0.0 0.0"/>
+        <geometry>
+            <sphere radius="${caster_radius}"/>
+        </geometry>
+    </collision>
+    <xacro:sphere_inertial
+        mass="${caster_mass}"
+        radius="${caster_radius}"
+        origin_xyz="0.0 0.0 0.0"/>
+</link>
+<joint name="caster_joint" type="fixed">
+    <parent link="base_link"/>
+    <child link="caster_link"/>
+    <origin
+        xyz="${caster_x_offset} 0.0 ${caster_radius}"
+        rpy="0.0 0.0 0.0"/>
+</joint>
     <!-- ================================================== -->
     <!-- Lidar                                              -->

Commit message: Week 3: Gazebo Sim Base

File: src/robot_description/urdf/robot.urdf.xacro (robot description, xacro)
@@ -243,8 +243,32 @@
         name="left"
         y_position="${wheel_separation / 2.0}"/>
+    <gazebo reference="left_wheel_link">
+        <collision>
+            <surface>
+                <friction>
+                    <ode>
+                        <mu>1.0</mu>
+                        <mu2>1.0</mu2>
+                    </ode>
+                </friction>
+            </surface>
+        </collision>
+    </gazebo>
     <!-- Right wheel -->
     <xacro:wheel
         name="right"
         y_position="${-wheel_separation / 2.0}"/>
+    <gazebo reference="right_wheel_link">
+        <collision>
+            <surface>
+                <friction>
+                    <ode>
+                        <mu>1.0</mu>
+                        <mu2>1.0</mu2>
+                    </ode>
+                </friction>
+            </surface>
+        </collision>
+    </gazebo>
 <!-- ================================================== -->
 <!-- Rear caster wheel                                  -->
@@ -283,6 +307,50 @@
 </joint>
     <!-- ================================================== -->
+    <!-- Gazebo Lidar Sensor                                -->
+    <!-- ================================================== -->
+    <gazebo reference="laser_frame">
+        <sensor name="gpu_lidar" type="gpu_lidar">
+            <!-- Sensor pose relative to laser_frame -->
+            <pose>0 0 0 0 0 0</pose>
+            <!-- Keep publishing while simulation is running -->
+            <always_on>true</always_on>
+            <!-- Scan frequency -->
+            <update_rate>10.0</update_rate>
+            <!-- Gazebo Transport topic -->
+            <topic>/scan</topic>
+            <!-- Show rays in Gazebo GUI -->
+            <visualize>true</visualize>
+            <lidar>
+                <scan>
+                    <horizontal>
+                        <!-- Number of laser beams -->
+                        <samples>360</samples>
+                        <!-- Usually keep resolution at 1 -->
+                        <resolution>1.0</resolution>
+                        <!-- -180 degrees -->
+                        <min_angle>-${pi}</min_angle>
+                        <!-- +180 degrees -->
+                        <max_angle>${pi}</max_angle>
+                    </horizontal>
+                </scan>
+                <range>
+                    <min>0.10</min>
+                    <max>12.0</max>
+                    <resolution>0.01</resolution>
+                </range>
+                <noise>
+                    <type>gaussian</type>
+                    <mean>0.0</mean>
+                    <stddev>0.01</stddev>
+                </noise>
+            </lidar>
+        </sensor>
+    </gazebo>
+    <!-- ================================================== -->
     <!-- Lidar                                              -->
     <!-- ================================================== -->
+    <gazebo reference="laser_joint">
+        <preserveFixedJoint>true</preserveFixedJoint>
+    </gazebo>
     <link name="laser_frame">
         <visual>

Commit message: feat: Week4 ROS2 Controller

File: src/robot_description/urdf/robot.urdf.xacro (robot description, xacro)
@@ -27,4 +27,6 @@
     <xacro:property name="lidar_z_offset" value="0.25"/>
     <xacro:property name="lidar_mass" value="0.2"/>
+    <!-- Gazebo controller -->
+    <xacro:property name="controllers_file" default="" />
     <!-- ================================================== -->
     <!-- Gazebo DiffDrive System                            -->
@@ -32,26 +34,7 @@
     <gazebo>
         <plugin
-            filename="gz-sim-diff-drive-system"
-            name="gz::sim::systems::DiffDrive">
-            <!-- Wheel joints -->
-            <left_joint>left_wheel_joint</left_joint>
-            <right_joint>right_wheel_joint</right_joint>
-            <!-- Robot geometry -->
-            <wheel_separation>${wheel_separation}</wheel_separation>
-            <wheel_radius>${wheel_radius}</wheel_radius>
-            <!-- Gazebo Transport topics -->
-            <topic>/cmd_vel</topic>
-            <odom_topic>/odom</odom_topic>
-            <!-- Odometry -->
-            <odom_publish_frequency>50</odom_publish_frequency>
-            <frame_id>odom</frame_id>
-            <child_frame_id>base_link</child_frame_id>
-            <!-- Motion limits -->
-            <max_linear_velocity>1.0</max_linear_velocity>
-            <min_linear_velocity>-1.0</min_linear_velocity>
-            <max_angular_velocity>2.0</max_angular_velocity>
-            <min_angular_velocity>-2.0</min_angular_velocity>
-            <max_linear_acceleration>1.0</max_linear_acceleration>
-            <max_angular_acceleration>2.0</max_angular_acceleration>
+            filename="libgz_ros2_control-system.so"
+            name="gz_ros2_control::GazeboSimROS2ControlPlugin">
+            <parameters>$(arg controllers_file)</parameters>
         </plugin>
     </gazebo>
@@ -271,4 +254,24 @@
         </collision>
     </gazebo>
+    <ros2_control name="GazeboSimSystem" type="system">
+        <hardware>
+            <plugin>gz_ros2_control/GazeboSimSystem</plugin>
+        </hardware>
+        <!-- left and right interface is here -->
+        <joint name="left_wheel_joint">
+            <!-- One command interface -->
+            <command_interface name="velocity"/>
+            <!-- Two state interface -->
+            <state_interface name="position"/>
+            <state_interface name="velocity"/>
+        </joint>
+        <joint name="right_wheel_joint">
+            <!-- One command interface -->
+            <command_interface name="velocity"/>
+            <!-- Two state interface -->
+            <state_interface name="position"/>
+            <state_interface name="velocity"/>
+        </joint>
+    </ros2_control>
 <!-- ================================================== -->
 <!-- Rear caster wheel                                  -->

Commit message: Week 7: Slam_toolbox

File: src/robot_description/urdf/robot.urdf.xacro (robot description, xacro)
@@ -174,4 +174,13 @@
             origin_xyz="0.0 0.0 ${base_center_z}"/>
     </link>
+    <!-- ================================================== -->
+    <!-- Base Footprint (地面投影点, slam_toolbox 默认要找它) -->
+    <!-- ================================================== -->
+    <link name="base_footprint"/>
+    <joint name="base_footprint_joint" type="fixed">
+        <parent link="base_link"/>
+        <child link="base_footprint"/>
+        <origin xyz="0.0 0.0 0.0" rpy="0.0 0.0 0.0"/>
+    </joint>
     <!-- ================================================== -->
     <!-- Wheel Macro                                        -->
