Commit message: Virtual Mobile Robot Version-0.9 Rebuild files and add README

File: src/robot_description/urdf/robot.urdf.xacro (robot description, xacro)
@@ -1,15 +1,22 @@
 <?xml version="1.0"?>
+<!--
+robot.urdf.xacro
+内含xacro写法, 但是不完全, 后续可以继续修改, 使文件更加简洁
+内容:
+机器人的形态及 Gazebo 插件, controller 插件
+-->
+<!-- xacro 声明 -->
 <robot
     xmlns:xacro="http://www.ros.org/wiki/xacro"
     name="virtual_mobile_robot">
-    <!-- ================================================== -->
-    <!-- Parameters                                         -->
-    <!-- ================================================== -->
-    <!-- Base -->
+    <!-- ==================================================  -->
+    <!-- 机器人参数                                           -->
+    <!-- ==================================================  -->
+    <!-- 本体 -->
     <xacro:property name="base_length" value="0.5"/>
     <xacro:property name="base_width" value="0.3"/>
     <xacro:property name="base_height" value="0.15"/>
     <xacro:property name="base_mass" value="5.0"/>
-    <!-- Wheels -->
+    <!-- 左右轮 -->
     <xacro:property name="wheel_radius" value="0.08"/>
     <xacro:property name="wheel_width" value="0.04"/>
@@ -17,9 +24,9 @@
     <xacro:property name="wheel_x_offset" value="0.05"/>
     <xacro:property name="wheel_mass" value="0.5"/>
-    <!-- Caster wheel -->
+    <!-- 万向轮 -->
     <xacro:property name="caster_radius" value="0.04"/>
     <xacro:property name="caster_x_offset" value="-0.20"/>
     <xacro:property name="caster_mass" value="0.1"/>
-    <!-- Lidar -->
+    <!-- 雷达 -->
     <xacro:property name="lidar_radius" value="0.05"/>
     <xacro:property name="lidar_height" value="0.04"/>
@@ -29,7 +36,5 @@
     <!-- Gazebo controller -->
     <xacro:property name="controllers_file" default="" />
-    <!-- ================================================== -->
-    <!-- Gazebo DiffDrive System                            -->
-    <!-- ================================================== -->
+    <!-- 全局 Gazebo 插件声明 -->
     <gazebo>
         <plugin
@@ -40,11 +45,9 @@
     </gazebo>
     <!--
-        base_link 位于地面中心附近。
+        base_link 高度
         轮子中心高度：
         wheel_radius = 0.08
         车体中心高度：
-        wheel_radius + base_height / 2
-        = 0.08 + 0.075
-        = 0.155
+        wheel_radius + base_height / 2 = 0.155
     -->
     <xacro:property
@@ -52,5 +55,5 @@
         value="${wheel_radius + base_height / 2.0}"/>
     <!-- ================================================== -->
-    <!-- Inertial Macros                                    -->
+    <!-- 惯性宏                                              -->
     <!-- ================================================== -->
     <!--
@@ -78,5 +81,4 @@
     </xacro:macro>
     <!--
-        Y 轴圆柱惯性宏
         适用于左右轮。
         圆柱轴线沿 Y 轴。
@@ -100,5 +102,4 @@
     </xacro:macro>
     <!--
-        Z 轴圆柱惯性宏
         适用于激光雷达外壳。
         圆柱轴线沿 Z 轴。
@@ -123,5 +124,4 @@
     <!--
     万向轮惯性宏
-    Sphere inertial macro
     -->
     <xacro:macro
@@ -143,5 +143,5 @@
     </xacro:macro>
     <!-- ================================================== -->
-    <!-- Base Link                                          -->
+    <!-- 车体定义                                             -->
     <!-- ================================================== -->
     <link name="base_link">
@@ -184,5 +184,5 @@
     </joint>
     <!-- ================================================== -->
-    <!-- Wheel Macro                                        -->
+    <!-- 两轮宏                                              -->
     <!-- ================================================== -->
     <xacro:macro name="wheel" params="name y_position">
@@ -231,4 +231,5 @@
         </joint>
     </xacro:macro>
+    <!-- 两侧轮子的定义 -->
     <!-- Left wheel -->
     <xacro:wheel
@@ -263,4 +264,7 @@
         </collision>
     </gazebo>
+    <!-- ================================================== -->
+    <!-- ROS2 control 接口声明                               -->
+    <!-- ================================================== -->
     <ros2_control name="GazeboSimSystem" type="system">
         <hardware>
@@ -283,70 +287,69 @@
         </joint>
     </ros2_control>
-<!-- ================================================== -->
-<!-- Rear caster wheel                                  -->
-<!-- ================================================== -->
-<link name="caster_link">
-    <visual>
+    <!-- ================================================== -->
+    <!-- Rear caster wheel                                  -->
+    <!-- ================================================== -->
+    <link name="caster_link">
+        <visual>
+            <origin
+                xyz="0.0 0.0 0.0"
+                rpy="0.0 0.0 0.0"/>
+            <geometry>
+                <sphere radius="${caster_radius}"/>
+            </geometry>
+            <material name="caster_gray">
+                <color rgba="0.25 0.25 0.25 1.0"/>
+            </material>
+        </visual>
+        <collision>
+            <origin
+                xyz="0.0 0.0 0.0"
+                rpy="0.0 0.0 0.0"/>
+            <geometry>
+                <sphere radius="${caster_radius}"/>
+            </geometry>
+        </collision>
+        <xacro:sphere_inertial
+            mass="${caster_mass}"
+            radius="${caster_radius}"
+            origin_xyz="0.0 0.0 0.0"/>
+    </link>
+    <joint name="caster_joint" type="fixed">
+        <parent link="base_link"/>
+        <child link="caster_link"/>
         <origin
-            xyz="0.0 0.0 0.0"
+            xyz="${caster_x_offset} 0.0 ${caster_radius}"
             rpy="0.0 0.0 0.0"/>
-        <geometry>
-            <sphere radius="${caster_radius}"/>
-        </geometry>
-        <material name="caster_gray">
-            <color rgba="0.25 0.25 0.25 1.0"/>
-        </material>
-    </visual>
-    <collision>
-        <origin
-            xyz="0.0 0.0 0.0"
-            rpy="0.0 0.0 0.0"/>
-        <geometry>
-            <sphere radius="${caster_radius}"/>
-        </geometry>
-    </collision>
-    <xacro:sphere_inertial
-        mass="${caster_mass}"
-        radius="${caster_radius}"
-        origin_xyz="0.0 0.0 0.0"/>
-</link>
-<joint name="caster_joint" type="fixed">
-    <parent link="base_link"/>
-    <child link="caster_link"/>
-    <origin
-        xyz="${caster_x_offset} 0.0 ${caster_radius}"
-        rpy="0.0 0.0 0.0"/>
-</joint>
-    <!-- ================================================== -->
-    <!-- Gazebo Lidar Sensor                                -->
+    </joint>
+    <!-- ================================================== -->
+    <!-- Gazebo 雷达传感器                                  -->
     <!-- ================================================== -->
     <gazebo reference="laser_frame">
         <sensor name="gpu_lidar" type="gpu_lidar">
-            <!-- specified frame name -->
-            <!-- <frame_id>laser_frame</frame_id> -->
+            <!-- 雷达frame的名字 -->
             <gz_frame_id>laser_frame</gz_frame_id>
-            <!-- Sensor pose relative to laser_frame -->
+            <!-- 雷达传感器和frame的位置关系 -->
             <pose>0 0 0 0 0 0</pose>
-            <!-- Keep publishing while simulation is running -->
+            <!-- 扫描时持续发布 -->
             <always_on>true</always_on>
-            <!-- Scan frequency -->
+            <!-- 扫描频率 Hz -->
             <update_rate>10.0</update_rate>
-            <!-- Gazebo Transport topic -->
+            <!-- 雷达发布topic -->
             <topic>/scan</topic>
-            <!-- Show rays in Gazebo GUI -->
+            <!-- 在 Gazebo 中展现雷达射线 -->
             <!-- <visualize>true</visualize> -->
             <lidar>
                 <scan>
                     <horizontal>
-                        <!-- Number of laser beams -->
+                        <!-- 雷达射线条数 -->
                         <samples>360</samples>
                         <!-- Usually keep resolution at 1 -->
                         <resolution>1.0</resolution>
-                        <!-- -180 degrees -->
+                        <!-- 角度值范围 360° -->
                         <min_angle>-${pi}</min_angle>
-                        <!-- +180 degrees -->
                         <max_angle>${pi}</max_angle>
                     </horizontal>
                 </scan>
+                <!-- 雷达探测距离范围 -->
                 <range>
                     <min>0.10</min>
